File: Hardware/CAD/PCB/V-Arc/V-Arc.kicad_pcb (KiCad board)
At the start: 2 copper layers, 200 x 100 mm, 94 parts, among them J1 USB_C_Receptacle_USB2.0_16P, J2 Conn_01x02, J3 AudioJack2_SwitchT, J4 AudioJack2, J5 AudioJack3, J6 AudioJack2, SW1 SW_SPDT, SW10 SW_Push, SW11 SW_Push, SW12 SW_SPDT, SW2 SW_SPDT, SW3 SW_SPDT, SW4 SW_SPDT, SW5 SW_SPDT, SW6 SW_SPDT, SW7 SW_Push, SW8 SW_SPDT_MSM, SW9 SW_SPDT, U1 BQ24072RGT, U2 MT3608, U3 MT3608, U4 MAX1044, U5 TL072, U6 Daisy_Seed, U7 XIAO-ESP32-S3-SMD, U8 ER_OLEDM0.91_1x-I2C, U9 TL072

Commit message: Finished PCB Layout
Parts:
- removed C26: 10 nF, Capacitor_SMD:C_0805_2012Metric
- removed SW11: SW_Push, Button_Switch_THT:SW_PUSH-12mm_Wuerth-430476085716
- RV6: footprint Potentiometer_THT:Potentiometer_Bourns_PTV09A-1_Single_Vertical -> Potentiometer_THT:Potentiometer_Alpha_RD902F-40-00D_Dual_Vertical
- moved C23 150.5 mm to (96.5, 72.5)
- moved SW10 138.4 mm to (157.0, 92.8), turned to 90 degrees
- moved C18 133.8 mm to (134.0, 86.5), turned to 90 degrees
- moved SW8 132.4 mm to (136.2, 110.5), turned to 90 degrees
- moved C22 125.4 mm to (121.5, 72.5)
- moved C25 124.3 mm to (159.4, 95.7)
- moved NT1 109.1 mm to (184.5, 75.0), turned to 90 degrees
- moved C21 100.2 mm to (146.5, 72.5)
- moved U7 95.3 mm to (228.4, 100.5), turned to -90 degrees
- moved C29 91.4 mm to (220.5, 64.7), turned to 90 degrees
- moved U8 87.0 mm to (209.0, 82.4), turned to -90 degrees
- moved C28 86.4 mm to (226.0, 80.5), turned to 180 degrees
- moved J4 83.5 mm to (213.0, 48.3), turned to -90 degrees
- moved J5 82.4 mm to (245.0, 53.5), turned to 90 degrees
- moved RV6 82.3 mm to (236.7, 74.9)
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Connections:
- J2 pad MP: (no net) -> GNDD
- U7 pad 3: Net-(U7-D2) -> unconnected-(U7-D2-Pad3)
Routing:
- net GNDD: track 0.00 -> 31.2 mm, vias 0 -> 8
- net Net-(SW12-B): track 0.00 -> 20.0 mm, vias 0 -> 2
- net /Power Management/VBAT+: track 0.00 -> 19.2 mm
- net /Power Management/VBUS: track 0.00 -> 19.1 mm
- net /Power Management/VSYS: track 0.00 -> 19.0 mm
- net Net-(U1-TS): track 0.00 -> 9.56 mm
- net GNDA: track 0.00 -> 4.61 mm, vias 0 -> 2
- net Net-(U1-ISET): track 0.00 -> 2.86 mm
- net Net-(D2-K): track 0.00 -> 2.64 mm
- net Net-(U1-ILIM): track 0.00 -> 2.47 mm
- net Net-(J1-CC2): track 0.00 -> 2.32 mm
- net Net-(D3-A): track 0.00 -> 1.74 mm
- net Net-(U1-~{CHG}): track 0.00 -> 1.72 mm
- net Net-(J1-CC1): track 0.00 -> 1.64 mm
- net Net-(D1-A): track 0.00 -> 1.49 mm
- added copper zone on B.Cu, net GNDA
- added copper zone on B.Cu, net GNDD

Commit message: Wired and Connected some zones
Routing:
- net /Analog Front End/+9V: track 0.00 -> 131.8 mm
- net /Daisy Seed Core/+3.3V: track 0.00 -> 124.0 mm
- net Net-(U6-D19): track 0.00 -> 99.9 mm
- net /Analog Front End/-9V: track 0.00 -> 95.7 mm, vias 0 -> 2
- net /Daisy Seed Core/+5V: track 0.00 -> 84.1 mm, vias 0 -> 4
- net Net-(U6-D18): track 0.00 -> 71.9 mm
- net GNDD: track 31.2 -> 100.3 mm, vias 8 -> 46
- net /Analog Front End/AUDIO_IN_ANALOG: track 0.00 -> 52.3 mm
- net Net-(U6-D17): track 0.00 -> 46.9 mm
- net GNDA: track 4.61 -> 41.8 mm, vias 2 -> 14
- net Net-(SW1-B): track 0.00 -> 25.2 mm
- net Net-(U6-D16): track 0.00 -> 22.6 mm
- net Net-(U6-D15): track 0.00 -> 21.7 mm
- net /Power Management/VSYS: track 19.0 -> 31.5 mm
- net Net-(C14-Pad2): track 0.00 -> 11.8 mm
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
Commit message: Finished PCB
Parts:
- moved NT1 98.7 mm to (86.0, 80.5), turned to 0 degrees
Connections:
- J2 pad MP: GNDD -> (no net)
- RV6 pad : GNDA -> (no net)
- SW4 pad 1: unconnected-(SW4-A-Pad1) -> Net-(SW4-A)
- U6 pad 4: Net-(SW4-C) -> Net-(SW4-A)
Routing:
- net /Daisy Seed Core/+5V: track 84.1 -> 246.0 mm
- net /Daisy Seed Core/AUDIO_OUT_ANALOG_L: track 0.00 -> 119.6 mm
- net Net-(U6-D6): track 0.00 -> 117.9 mm
- net /Daisy Seed Core/DSP_UART_RX: track 0.00 -> 113.9 mm
- net /Daisy Seed Core/DSP_UART_TX: track 0.00 -> 107.0 mm, vias 0 -> 2
- net Net-(U7-D3): track 0.00 -> 102.7 mm, vias 0 -> 2
- net /Daisy Seed Core/AUDIO_OUT_ANALOG_R: track 0.00 -> 102.3 mm
- net GNDD: track 100.3 -> 198.4 mm, vias 46 -> 68
- net Net-(SW9-A): track 0.00 -> 93.0 mm
- net Net-(SW4-A): track 0.00 -> 77.1 mm
- net Net-(SW6-A): track 0.00 -> 64.6 mm
- net /Xiao ESP Core/OUT_L_FINAL: track 0.00 -> 52.8 mm
- net /Xiao ESP Core/XiaoV: track 0.00 -> 48.0 mm, vias 0 -> 2
- net Net-(SW3-A): track 0.00 -> 46.0 mm
- net Net-(SW5-A): track 0.00 -> 34.5 mm
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
Commit message: Added BOM
Parts:
- removed J6: AudioJack2, Connector_Audio:Jack_3.5mm_CUI_SJ1-3513N_Horizontal
- added R21: 10 kΩ, Resistor_SMD:R_0805_2012Metric, F.Cu at (225.0, 58.0)
- added R22: 10 kΩ, Resistor_SMD:R_0805_2012Metric, F.Cu at (225.0, 56.0)
- C14: footprint Capacitor_SMD:CP_Elec_6.3x5.4 -> Capacitor_SMD:C_0805_2012Metric
- J3, J4: footprint Connector_Audio:Jack_3.5mm_CUI_SJ1-3513N_Horizontal -> Connector_Audio:Jack_6.35mm_Neutrik_NMJ4HCD2_Horizontal
- moved J4 17.6 mm to (204.9, 63.9), turned to 90 degrees
- moved J3 15.1 mm to (66.4, 129.6), turned to 180 degrees
- moved R20 11.9 mm to (232.2, 59.5)
- moved C29 7.15 mm to (227.7, 64.6)
- moved C14 4.61 mm to (73.0, 133.0)
- moved C19 2.50 mm to (194.0, 72.5)
- moved RV5 2.00 mm to (198.0, 70.0)
- moved R17 1.45 mm to (224.9, 69.3)
- moved C30 0.72 mm to (236.0, 64.9)
- moved R19 0.72 mm to (235.9, 58.1)
Connections:
- J4 pad T: /Xiao ESP Core/OUT_L_FINAL -> Net-(J4-PadT)
Routing:
- net GNDA: track 70.5 -> 43.0 mm, vias 25 -> 22
- net /Xiao ESP Core/OUT_L_FINAL: track 52.8 -> 25.7 mm
- net Net-(J4-PadT): track 0.00 -> 23.7 mm
- net GNDD: track 198.4 -> 193.1 mm, vias 68 -> 64
- net Net-(C14-Pad2): track 11.8 -> 7.02 mm
- net /Xiao ESP Core/OUT_R_FINAL: track 23.0 -> 27.4 mm
- net /Daisy Seed Core/+5V: track 246.0 -> 248.9 mm
- net Net-(SW1-B): track 25.2 -> 23.0 mm
- net /Daisy Seed Core/+3.3V: track 124.0 -> 122.1 mm
- net Net-(C29-Pad1): track 2.83 -> 4.47 mm
- net Net-(U6-D19): track 99.9 -> 99.1 mm
- net Net-(U9A--): track 3.99 -> 4.72 mm
- net Net-(C30-Pad1): track 2.79 -> 3.51 mm
- net /Analog Front End/+9V: track 131.8 -> 132.2 mm, vias 0 -> 2
